Commit message: trying the comp objective instead

File: urdf/brick.urdf (robot description, URDF)
Before this commit: robot Brick, 2 links, 1 joints
Links:
- added link contact2, mass 1e-12; collision sphere radius=0; visual sphere radius=.05
- added link contact3, mass 1e-12; collision sphere radius=0; visual sphere radius=.05
- added link contact4, mass 1e-12; collision sphere radius=0; visual sphere radius=.05
- added link floor; collision box size=2.2 2.2 0.1; collision plane normal=0 0 1
- link contact1: geometry collision sphere radius=0; visual sphere radius=.05
Joints:
- added joint contact2_to_brick: type fixed, parent brick, child contact2, origin xyz=.5 -.5 -.5
- added joint contact3_to_brick: type fixed, parent brick, child contact3, origin xyz=-.5 -.5 -.5
- added joint contact4_to_brick: type fixed, parent brick, child contact4, origin xyz=-.5 .5 -.5
- added joint floor_to_brick: type fixed, parent floor, child brick, origin xyz=0 0 1
- joint contact1_to_brick: origin xyz=0. 0. -.5 -> xyz=.5 .5 -.5
