Commit message: wip: reversediff with tapes

File: urdf/ball.urdf (robot description, URDF)
Before this commit: robot Ball, 2 links, 1 joints
Links:
- link floor: geometry visual box size=2.5 2.5 0.1

Commit message: wip: major refactor

File: urdf/ball.urdf (robot description, URDF)
Before this commit: robot Ball, 2 links, 1 joints
Joints:
- joint floor_to_ball: type fixed -> floating
