Commit message: franka urdf

File: urdf/panda/panda_arm.urdf (robot description, URDF)
Before this commit: robot panda, 9 links, 8 joints
Links:
- link panda_link0: mass None -> 0.1; geometry visual mesh filename=../urdf/panda/meshes/link0.obj
- link panda_link1: mass None -> 0.1; geometry visual mesh filename=../urdf/panda/meshes/link1.obj
- link panda_link2: mass None -> 0.1; geometry visual mesh filename=../urdf/panda/meshes/link2.obj
- link panda_link3: mass None -> 0.1; geometry visual mesh filename=../urdf/panda/meshes/link3.obj
- link panda_link4: mass None -> 0.1; geometry visual mesh filename=../urdf/panda/meshes/link4.obj
- link panda_link5: mass None -> 0.1; geometry visual mesh filename=../urdf/panda/meshes/link5.obj
- link panda_link6: mass None -> 0.1; geometry visual mesh filename=../urdf/panda/meshes/link6.obj
- link panda_link7: mass None -> 0.1; geometry visual mesh filename=../urdf/panda/meshes/link7.obj
- link panda_link8: mass None -> 0.1; geometry visual sphere radius=.025
Joints:
- joint panda_joint1: axis 0 0 1 -> 0 1 0; limit lower=-2.8973 upper=2.8973 effort=87 velocity=2.1750 -> (none); origin xyz=0 0 0.333 rpy=0 0 0 -> xyz=0 0 0.333 rpy=1.57079632679 0 0
- joint panda_joint2: axis 0 0 1 -> 0 1 0; limit lower=-1.7628 upper=1.7628 effort=87 velocity=2.1750 -> (none)
- joint panda_joint3: axis 0 0 1 -> 0 1 0; limit lower=-2.8973 upper=2.8973 effort=87 velocity=2.1750 -> (none); origin xyz=0 -0.316 0 rpy=1.57079632679 0 0 -> xyz=0 0 0.316 rpy=1.57079632679 0 0
- joint panda_joint4: axis 0 0 1 -> 0 1 0; limit lower=-3.0718 upper=-0.0698 effort=87 velocity=2.1750 -> (none)
- joint panda_joint5: axis 0 0 1 -> 0 1 0; limit lower=-2.8973 upper=2.8973 effort=12 velocity=2.6100 -> (none); origin xyz=-0.0825 0.384 0 rpy=-1.57079632679 0 0 -> xyz=-0.0825 0 -0.384 rpy=-1.57079632679 0 0
- joint panda_joint6: axis 0 0 1 -> 0 1 0; limit lower=-0.0175 upper=3.7525 effort=12 velocity=2.6100 -> (none)
- joint panda_joint7: axis 0 0 1 -> 0 1 0; limit lower=-2.8973 upper=2.8973 effort=12 velocity=2.6100 -> (none)
- joint panda_joint8: axis 0 0 0 -> (none); origin xyz=0 0 0.107 rpy=0 0 0 -> xyz=0 .1 0 rpy=0 0 0

Commit message: wip simulation to get the regression data

File: urdf/panda/panda_arm.urdf (robot description, URDF)
Before this commit: robot panda, 9 links, 8 joints
Links:
- link panda_link0: mass 0.1 -> 1.
- link panda_link1: mass 0.1 -> 1.
- link panda_link2: mass 0.1 -> 1.
- link panda_link3: mass 0.1 -> 1.
- link panda_link4: mass 0.1 -> 1.
- link panda_link5: mass 0.1 -> 1.
- link panda_link6: mass 0.1 -> 1.
- link panda_link7: mass 0.1 -> 1.
- link panda_link8: mass 0.1 -> 1.

File: urdf/panda/panda_arm_box.urdf (robot description, URDF)
Before this commit: robot panda, 11 links, 10 joints
Links:
- link box: mass .00001 -> .001
- link panda_link0: mass 0.1 -> 1.
- link panda_link1: mass 0.1 -> 1.
- link panda_link2: mass 0.1 -> 1.
- link panda_link3: mass 0.1 -> 1.
- link panda_link4: mass 0.1 -> 1.
- link panda_link5: mass 0.1 -> 1.
- link panda_link6: mass 0.1 -> 1.
- link panda_link7: mass 0.1 -> 1.
- link panda_link8: mass 0.1 -> 1.
