Commit message: wip robust franka trajopt

File: urdf/panda/panda_arm_plate.urdf (robot description, URDF)
Before this commit: robot panda, 9 links, 8 joints
Joints:
- joint panda_joint8: origin xyz=0 0.11 0 rpy=1.57079632679 0 0 -> xyz=0 0 0 rpy=0 0 0

Commit message: working robust control example

File: urdf/panda/panda_arm_plate.urdf (robot description, URDF)
Before this commit: robot panda, 9 links, 8 joints
Joints:
- joint panda_joint8: origin xyz=0 0 0 rpy=0 0 0 -> xyz=0 0.11 0 rpy=-1.57079632679 0 0

Commit message: decent run on the robust traj opt - keeping in case

File: urdf/panda/panda_arm_plate.urdf (robot description, URDF)
Before this commit: robot panda, 9 links, 8 joints
Links:
- link panda_link8: geometry visual box size=.35 .35 .01
