Commit message: explicit contact with panda box

File: urdf/panda/panda_arm_box.urdf (robot description, URDF)
Before this commit: robot panda, 12 links, 11 joints
Links:
- removed link contact1
- link box: mass 1. -> .00001; geometry collision sphere radius=0; collision sphere radius=0
- link floor: geometry visual box size=10 2 0.1
Joints:
- removed joint contact1_to_box
- joint floor_to_box: origin xyz=1 0 .25 -> xyz=0 0 0

Commit message: working contact simulation for parameter regression

File: urdf/panda/panda_arm_box.urdf (robot description, URDF)
Before this commit: robot panda, 11 links, 10 joints
Links:
- link box: mass .001 -> 10.

Commit message: wip: bigger example parameter regression

File: urdf/panda/panda_arm_box.urdf (robot description, URDF)
Before this commit: robot panda, 11 links, 10 joints
Links:
- link floor: geometry visual box size=4 3 0.1

Commit message: wip: trying to move cn to lower problem

File: urdf/panda/panda_arm_box.urdf (robot description, URDF)
Before this commit: robot panda, 11 links, 10 joints
Joints:
- joint floor_to_box: type fixed -> floating
