Commit message: wip: trajopt for littledog

File: urdf/little_dog/little_dog.urdf (robot description, URDF)
Before this commit: robot little_dog, 14 links, 13 joints
Links:
- link back_left_lower_leg: geometry collision sphere radius=0; visual mesh filename=/Users/blandry/.julia/dev/Bilevel/urdf/little_dog/meshes/ba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
- link back_right_lower_leg: geometry collision sphere radius=0; visual mesh filename=/Users/blandry/.julia/dev/Bilevel/urdf/little_dog/meshes/ba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
- link front_left_lower_leg: geometry collision sphere radius=0; visual mesh filename=/Users/blandry/.julia/dev/Bilevel/urdf/little_dog/meshes/fr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
- link front_right_lower_leg: geometry collision sphere radius=0; visual mesh filename=/Users/blandry/.julia/dev/Bilevel/urdf/little_dog/meshes/fr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

Commit message: urdf path

File: urdf/little_dog/little_dog.urdf (robot description, URDF)
Before this commit: robot little_dog, 14 links, 13 joints
Links:
- link back_left_lower_leg: geometry collision sphere radius=0; visual mesh filename=/home/blandry/.julia/dev/Bilevel/urdf/little_dog/meshes/bac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
- link back_left_upper_leg: geometry visual mesh filename=/home/blandry/.julia/dev/Bilevel/urdf/little_dog/meshes/bac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
- link back_right_lower_leg: geometry collision sphere radius=0; visual mesh filename=/home/blandry/.julia/dev/Bilevel/urdf/little_dog/meshes/bac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
- link back_right_upper_leg: geometry visual mesh filename=/home/blandry/.julia/dev/Bilevel/urdf/little_dog/meshes/bac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
- link body: geometry visual mesh filename=/home/blandry/.julia/dev/Bilevel/urdf/little_dog/meshes/bod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
- link front_left_lower_leg: geometry collision sphere radius=0; visual mesh filename=/home/blandry/.julia/dev/Bilevel/urdf/little_dog/meshes/fro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
- link front_left_upper_leg: geometry visual mesh filename=/home/blandry/.julia/dev/Bilevel/urdf/little_dog/meshes/fro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
- link front_right_lower_leg: geometry collision sphere radius=0; visual mesh filename=/home/blandry/.julia/dev/Bilevel/urdf/little_dog/meshes/fro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
- link front_right_upper_leg: geometry visual mesh filename=/home/blandry/.julia/dev/Bilevel/urdf/little_dog/meshes/fro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

Commit message: mesh path

File: urdf/little_dog/little_dog.urdf (robot description, URDF)
Before this commit: robot little_dog, 14 links, 13 joints
Links:
- link back_left_lower_leg: geometry collision sphere radius=0; visual mesh filename=/Users/blandry/.julia/dev/Bilevel/urdf/little_dog/meshes/ba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
- link back_left_upper_leg: geometry visual mesh filename=/Users/blandry/.julia/dev/Bilevel/urdf/little_dog/meshes/ba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
- link back_right_lower_leg: geometry collision sphere radius=0; visual mesh filename=/Users/blandry/.julia/dev/Bilevel/urdf/little_dog/meshes/ba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
- link back_right_upper_leg: geometry visual mesh filename=/Users/blandry/.julia/dev/Bilevel/urdf/little_dog/meshes/ba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
- link body: geometry visual mesh filename=/Users/blandry/.julia/dev/Bilevel/urdf/little_dog/meshes/bo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
- link front_left_lower_leg: geometry collision sphere radius=0; visual mesh filename=/Users/blandry/.julia/dev/Bilevel/urdf/little_dog/meshes/fr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
- link front_left_upper_leg: geometry visual mesh filename=/Users/blandry/.julia/dev/Bilevel/urdf/little_dog/meshes/fr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
- link front_right_lower_leg: geometry collision sphere radius=0; visual mesh filename=/Users/blandry/.julia/dev/Bilevel/urdf/little_dog/meshes/fr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
- link front_right_upper_leg: geometry visual mesh filename=/Users/blandry/.julia/dev/Bilevel/urdf/little_dog/meshes/fr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

Commit message: pining rbd.jl and small syntax fix

File: urdf/little_dog/little_dog.urdf (robot description, URDF)
Before this commit: robot little_dog, 14 links, 13 joints
Links:
- link back_left_lower_leg: geometry collision sphere radius=0; visual mesh filename=/home/blandry/Code/Bilevel.jl/urdf/little_dog/meshes/back_l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
- link back_left_upper_leg: geometry visual mesh filename=/home/blandry/Code/Bilevel.jl/urdf/little_dog/meshes/back_l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
- link back_right_lower_leg: geometry collision sphere radius=0; visual mesh filename=/home/blandry/Code/Bilevel.jl/urdf/little_dog/meshes/back_r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
- link back_right_upper_leg: geometry visual mesh filename=/home/blandry/Code/Bilevel.jl/urdf/little_dog/meshes/back_r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
- link body: geometry visual mesh filename=/home/blandry/Code/Bilevel.jl/urdf/little_dog/meshes/body.o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
- link front_left_lower_leg: geometry collision sphere radius=0; visual mesh filename=/home/blandry/Code/Bilevel.jl/urdf/little_dog/meshes/front_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
- link front_left_upper_leg: geometry visual mesh filename=/home/blandry/Code/Bilevel.jl/urdf/little_dog/meshes/front_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
- link front_right_lower_leg: geometry collision sphere radius=0; visual mesh filename=/home/blandry/Code/Bilevel.jl/urdf/little_dog/meshes/front_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
- link front_right_upper_leg: geometry visual mesh filename=/home/blandry/Code/Bilevel.jl/urdf/little_dog/meshes/front_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

File: urdf/little_dog/little_dog2d.urdf (robot description, URDF)
Before this commit: robot little_dog2d, 14 links, 13 joints
Links:
- link back_left_lower_leg: geometry collision sphere radius=0; visual mesh filename=/home/blandry/Code/Bilevel.jl/urdf/little_dog/meshes/back_l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
- link back_left_upper_leg: geometry visual mesh filename=/home/blandry/Code/Bilevel.jl/urdf/little_dog/meshes/back_l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
- link back_right_lower_leg: geometry collision sphere radius=0; visual mesh filename=/home/blandry/Code/Bilevel.jl/urdf/little_dog/meshes/back_r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
- link back_right_upper_leg: geometry visual mesh filename=/home/blandry/Code/Bilevel.jl/urdf/little_dog/meshes/back_r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
- link body: geometry visual mesh filename=/home/blandry/Code/Bilevel.jl/urdf/little_dog/meshes/body.o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
- link front_left_lower_leg: geometry collision sphere radius=0; visual mesh filename=/home/blandry/Code/Bilevel.jl/urdf/little_dog/meshes/front_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
- link front_left_upper_leg: geometry visual mesh filename=/home/blandry/Code/Bilevel.jl/urdf/little_dog/meshes/front_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
- link front_right_lower_leg: geometry collision sphere radius=0; visual mesh filename=/home/blandry/Code/Bilevel.jl/urdf/little_dog/meshes/front_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
- link front_right_upper_leg: geometry visual mesh filename=/home/blandry/Code/Bilevel.jl/urdf/little_dog/meshes/front_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
